File: pcb/emonpi3/emonPi3.kicad_sch (KiCad schematic)
At the start: 131 parts, among them CN1 CONN_03SCREW, CN2 CONN_03SCREW, CN3 CONN_03SCREW, J10 Conn_ARM_JTAG_SWD_10, J11 Conn_02x13_Odd_Even, J12 PINHD-1X9, J7 CONN_04PTH, J8 CONN_04PTH, J9 USB_C_Receptacle_USB2.0, SW1 SW_Push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

Commit message: * Swap SPI MOSI and !SS pins, incorrect in v0.1
Connections:
- net RFM_MOSI_UC: now also U3.32 (PA15); no longer U3.31 (PA14)
- net RFM_SEL_UC: now also U3.31 (PA14); no longer U3.32 (PA15)
Changed lines of the file:
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@@
     (effects (font (size 1.27 1.27)) (justify right bottom))
   )
-  (label "RFM_SEL_UC" (at 223.52 210.82 0) (fields_autoplaced)
+  (label "RFM_SEL_UC" (at 223.52 208.28 0) (fields_autoplaced)
     (effects (font (size 1.27 1.27)) (justify left bottom))
   )
@@
     (effects (font (size 1.2446 1.2446)) (justify left bottom))
   )
-  (label "RFM_MOSI_UC" (at 223.52 208.28 0) (fields_autoplaced)
+  (label "RFM_MOSI_UC" (at 223.52 210.82 0) (fields_autoplaced)
     (effects (font (size 1.27 1.27)) (justify left bottom))
   )

Commit message: * Move external interface disable pin. Remove USB sense.
Parts:
- removed R47, R48: 10K, Resistor_SMD:R_0603_1608Metric, symbol Device:R
Connections:
- net VUSB_SENSE is gone; now on net ~{DISABLE_EXT_INTF}: U3.38 (PA19)
- net ~{DISABLE_EXT_INTF}: now reaches J11.11 (Pin_11)
- no-connect marks 17 -> 16
Changed lines of the file:
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@@
   (junction (at 165.1 245.11) (diameter 0) (color 0 0 0 0)
   )
-  (junction (at 297.18 372.11) (diameter 0) (color 0 0 0 0)
-  )
   (junction (at 482.6 356.87) (diameter 0) (color 0 0 0 0)
   )
@@
   (no_connect (at 537.21 76.2))
   (no_connect (at 241.3 344.17))
-  (no_connect (at 406.4 64.77))
   (no_connect (at 537.21 73.66))
   (no_connect (at 419.1 64.77))
@@
     (stroke (width 0) (type default))
   )
+  (wire (pts (xy 384.81 64.77) (xy 406.4 64.77))
+    (stroke (width 0.1524) (type solid))
+  )
   (wire (pts (xy 220.98 93.98) (xy 220.98 104.14))
     (stroke (width 0) (type default))
@@
     (stroke (width 0) (type default))
   )
-  (wire (pts (xy 297.18 370.84) (xy 297.18 372.11))
-    (stroke (width 0) (type default))
-  )
   (wire (pts (xy 223.52 180.34) (xy 240.03 180.34))
     (stroke (width 0) (type default))
@@
     (stroke (width 0) (type default))
   )
-  (wire (pts (xy 297.18 372.11) (xy 297.18 373.38))
-    (stroke (width 0) (type default))
-  )
   (wire (pts (xy 544.83 312.42) (xy 544.83 314.96))
     (stroke (width 0) (type default))
@@
     (stroke (width 0) (type default))
   )
-  (wire (pts (xy 297.18 381) (xy 297.18 383.54))
-    (stroke (width 0) (type default))
-  )
   (wire (pts (xy 331.47 97.79) (xy 331.47 101.6))
     (stroke (width 0.1524) (type solid))
@@
     (stroke (width 0) (type default))
   )
-  (wire (pts (xy 297.18 360.68) (xy 297.18 363.22))
-    (stroke (width 0) (type default))
-  )
   (wire (pts (xy 82.55 76.2) (xy 82.55 80.01))
     (stroke (width 0) (type default))
@@
     (stroke (width 0) (type default))
   )
-  (wire (pts (xy 297.18 372.11) (xy 311.15 372.11))
-    (stroke (width 0) (type default))
-  )
   (wire (pts (xy 508 54.61) (xy 511.81 54.61))
     (stroke (width 0) (type default))
@@
     (effects (font (size 1.27 1.27)) (justify left bottom))
   )
+  (label "~{DISABLE_EXT_INTF}" (at 384.81 64.77 0) (fields_autoplaced)
+    (effects (font (size 1.27 1.27)) (justify left bottom))
+  )
   (label "UART_DBG_RX1" (at 431.8 152.4 0) (fields_autoplaced)
     (effects (font (size 1.27 1.27)) (justify left bottom))
@@
     (effects (font (size 1.27 1.27)) (justify right bottom))
   )
-  (label "VUSB_SENSE" (at 311.15 372.11 180) (fields_autoplaced)
-    (effects (font (size 1.27 1.27)) (justify right bottom))
-  )
   (label "VSENS1" (at 185.42 279.4 0) (fields_autoplaced)
     (effects (font (size 1.2446 1.2446)) (justify left bottom))
@@
     (effects (font (size 1.27 1.27)) (justify right bottom))
   )
-  (label "5V_USB" (at 297.18 360.68 0) (fields_autoplaced)
-    (effects (font (size 1.27 1.27)) (justify left bottom))
-  )
   (label "RFM_SEL" (at 440.69 69.85 180) (fields_autoplaced)
     (effects (font (size 1.2446 1.2446)) (justify right bottom))
@@
     (effects (font (size 1.27 1.27)) (justify left bottom))
   )
-  (label "VUSB_SENSE" (at 223.52 220.98 0) (fields_autoplaced)
+  (label "~{DISABLE_EXT_INTF}" (at 223.52 220.98 0) (fields_autoplaced)
     (effects (font (size 1.27 1.27)) (justify left bottom))
   )
@@
     )
   )
-  (symbol (lib_id "power:GND") (at 297.18 383.54 0) (unit 1)
-    (in_bom yes) (on_board yes) (dnp no) (fields_autoplaced)
-    (property "Reference" "#PWR040" (at 297.18 389.89 0)
-      (effects (font (size 1.27 1.27)) hide)
-    )
-    (property "Value" "GND" (at 297.18 388.62 0)
-      (effects (font (size 1.27 1.27)))
-    )
-    (property "Footprint" "" (at 297.18 383.54 0)
-      (effects (font (size 1.27 1.27)) hide)
-    )
-    (property "Datasheet" "" (at 297.18 383.54 0)
-      (effects (font (size 1.27 1.27)) hide)
-    )
-    (pin "1")
-    (instances
-      (project "emonPi3"
-        (path "/3a5f1087-1abe-4575-9313-bd86a5e03366"
-          (reference "#PWR040") (unit 1)
-        )
-      )
-    )
-  )
   (symbol (lib_id "Mechanical:Fiducial") (at 483.87 314.96 0) (unit 1)
     (in_bom no) (on_board yes) (dnp no)
@@
     )
   )
-  (symbol (lib_id "Device:R") (at 297.18 367.03 180) (unit 1)
-    (in_bom yes) (on_board yes) (dnp no)
-    (property "Reference" "R47" (at 298.45 364.49 0)
-      (effects (font (size 1.27 1.27)) (justify right bottom))
-    )
-    (property "Value" "10K" (at 298.45 367.03 0)
-      (effects (font (size 1.27 1.27)) (justify right))
-    )
-    (property "Footprint" "Resistor_SMD:R_0603_1608Metric" (at 298.958 367.03 90)
-      (effects (font (size 1.27 1.27)) hide)
-    )
-    (property "Datasheet" "~" (at 297.18 367.03 0)
-      (effects (font (size 1.27 1.27)) hide)
-    )
-    (pin "1")
-    (pin "2")
-    (instances
-      (project "emonPi3"
-        (path "/3a5f1087-1abe-4575-9313-bd86a5e03366"
-          (reference "R47") (unit 1)
-        )
-      )
-    )
-  )
   (symbol (lib_id "Device:R") (at 101.6 91.44 180) (unit 1)
     (in_bom yes) (on_board yes) (dnp no)
@@
         )
       )
-    )
-  )
-  (symbol (lib_id "Device:R") (at 297.18 377.19 180) (unit 1)
-    (in_bom yes) (on_board yes) (dnp no)
-    (property "Reference" "R48" (at 298.45 374.65 0)
-      (effects (font (size 1.27 1.27)) (justify right bottom))
-    )
-    (property "Value" "10K" (at 298.45 377.19 0)
-      (effects (font (size 1.27 1.27)) (justify right))
-    )
-    (property "Footprint" "Resistor_SMD:R_0603_1608Metric" (at 298.958 377.19 90)
-      (effects (font (size 1.27 1.27)) hide)
-    )
-    (property "Datasheet" "~" (at 297.18 377.19 0)
-      (effects (font (size 1.27 1.27)) hide)
-    )
-    (pin "1")
-    (pin "2")
-    (instances
-      (project "emonPi3"
-        (path "/3a5f1087-1abe-4575-9313-bd86a5e03366"
-          (reference "R48") (unit 1)
-        )
-      )

Commit message: * Change comparator from LMV331 to MCP6546
Parts:
- U6: value LMV331 -> MCP6456U
Other:
- note removed: "1M Burden resistors not populated Correct values should be choosen if using current output CT sensors."
- moved on the sheet: C9, R7
Changed lines of the file:
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@@
   (junction (at 372.11 323.85) (diameter 0) (color 0 0 0 0)
   )
-  (junction (at 73.66 364.49) (diameter 0) (color 0 0 0 0)
+  (junction (at 73.66 361.95) (diameter 0) (color 0 0 0 0)
   )
   (junction (at 374.65 175.26) (diameter 0) (color 0 0 0 0)
@@
     (stroke (width 0.1524) (type solid))
   )
-  (wire (pts (xy 46.99 364.49) (xy 63.5 364.49))
+  (wire (pts (xy 46.99 361.95) (xy 63.5 361.95))
     (stroke (width 0) (type default))
   )
@@
     (stroke (width 0) (type default))
   )
-  (wire (pts (xy 71.12 364.49) (xy 73.66 364.49))
+  (wire (pts (xy 71.12 361.95) (xy 73.66 361.95))
     (stroke (width 0) (type default))
   )
@@
     (stroke (width 0) (type default))
   )
-  (wire (pts (xy 73.66 364.49) (xy 73.66 367.03))
+  (wire (pts (xy 73.66 361.95) (xy 73.66 364.49))
     (stroke (width 0) (type default))
   )
@@
     (stroke (width 0.1524) (type solid))
   )
-  (wire (pts (xy 73.66 374.65) (xy 73.66 377.19))
+  (wire (pts (xy 73.66 372.11) (xy 73.66 374.65))
     (stroke (width 0) (type default))
   )
@@
     (stroke (width 0) (type default))
   )
-  (wire (pts (xy 73.66 364.49) (xy 90.17 364.49))
+  (wire (pts (xy 73.66 361.95) (xy 90.17 361.95))
     (stroke (width 0) (type default))
   )
@@
     (effects (font (size 1.27 1.27)) (justify left top))
   )
-  (text_box "Set ~{RPI_PRESENT} LOW on RasPi boot to indicate presence.\n\nThis will disable connected interfaces in the SAMD."
+  (text_box "Set ~{DISABLE_EXT_INTF} LOW on RasPi boot to indicate presence.\n\nThis will disable connected interfaces in the SAMD."
     (at 377.19 97.79 0) (size 35.56 11.43)
     (stroke (width 0) (type default))
@@
     (effects (font (size 1.27 1.27)) (justify left bottom))
   )
-  (text "1M Burden resistors not populated\nCorrect values should be choosen if\nusing current output CT sensors."
-    (at 13.97 140.97 0)
-    (effects (font (size 1.5 1.5)) (justify left bottom))
-  )
   (text "Voltage Reference Generation" (at 15.24 17.78 0)
     (effects (font (size 2 2) (thickness 0.4) bold) (justify left bottom))
@@
     (effects (font (size 1.27 1.27)) (justify right bottom))
   )
-  (label "ANALOG_INPUT" (at 46.99 364.49 0) (fields_autoplaced)
+  (label "ANALOG_INPUT" (at 46.99 361.95 0) (fields_autoplaced)
     (effects (font (size 1.27 1.27)) (justify left bottom))
   )
@@
     (effects (font (size 1.27 1.27)) (justify right bottom))
   )
-  (label "AIN_LPFILT" (at 90.17 364.49 180) (fields_autoplaced)
+  (label "AIN_LPFILT" (at 90.17 361.95 180) (fields_autoplaced)
     (effects (font (size 1.27 1.27)) (justify right bottom))
   )
@@
     )
   )
-  (symbol (lib_id "Device:C") (at 73.66 370.84 0) (unit 1)
+  (symbol (lib_id "Device:C") (at 73.66 368.3 0) (unit 1)
     (in_bom yes) (on_board yes) (dnp no)
-    (property "Reference" "C9" (at 76.2 369.57 0)
+    (property "Reference" "C9" (at 76.2 367.03 0)
       (effects (font (size 1.27 1.27)) (justify left bottom))
     )
-    (property "Value" "10n" (at 76.2 372.11 0)
+    (property "Value" "10n" (at 76.2 369.57 0)
       (effects (font (size 1.27 1.27)) (justify left bottom))
     )
-    (property "Footprint" "Capacitor_SMD:C_0603_1608Metric" (at 74.6252 374.65 0)
+    (property "Footprint" "Capacitor_SMD:C_0603_1608Metric" (at 74.6252 372.11 0)
       (effects (font (size 1.27 1.27)) hide)
     )
-    (property "Datasheet" "~" (at 73.66 370.84 0)
+    (property "Datasheet" "~" (at 73.66 368.3 0)
       (effects (font (size 1.27 1.27)) hide)
     )
@@
     )
   )
-  (symbol (lib_id "power:GND") (at 73.66 377.19 0) (unit 1)
+  (symbol (lib_id "power:GND") (at 73.66 374.65 0) (unit 1)
     (in_bom yes) (on_board yes) (dnp no) (fields_autoplaced)
-    (property "Reference" "#PWR06" (at 73.66 383.54 0)
+    (property "Reference" "#PWR06" (at 73.66 381 0)
       (effects (font (size 1.27 1.27)) hide)
     )
-    (property "Value" "GND" (at 73.66 382.27 0)
+    (property "Value" "GND" (at 73.66 379.73 0)
       (effects (font (size 1.27 1.27)))
     )
-    (property "Footprint" "" (at 73.66 377.19 0)
+    (property "Footprint" "" (at 73.66 374.65 0)
       (effects (font (size 1.27 1.27)) hide)
     )
-    (property "Datasheet" "" (at 73.66 377.19 0)
+    (property "Datasheet" "" (at 73.66 374.65 0)
       (effects (font (size 1.27 1.27)) hide)
     )
@@
     )
   )
-  (symbol (lib_id "Device:R") (at 67.31 364.49 270) (mirror x) (unit 1)
+  (symbol (lib_id "Device:R") (at 67.31 361.95 270) (mirror x) (unit 1)
     (in_bom yes) (on_board yes) (dnp no)
-    (property "Reference" "R7" (at 64.77 363.22 90)
+    (property "Reference" "R7" (at 64.77 360.68 90)
       (effects (font (size 1.27 1.27)) (justify left top))
     )
-    (property "Value" "3K3" (at 64.77 365.76 90)
+    (property "Value" "3K3" (at 64.77 363.22 90)
       (effects (font (size 1.27 1.27)) (justify left bottom))
     )
-    (property "Footprint" "Resistor_SMD:R_0603_1608Metric" (at 67.31 366.268 90)
+    (property "Footprint" "Resistor_SMD:R_0603_1608Metric" (at 67.31 363.728 90)
       (effects (font (size 1.27 1.27)) hide)
     )
-    (property "Datasheet" "~" (at 67.31 364.49 0)
+    (property "Datasheet" "~" (at 67.31 361.95 0)
       (effects (font (size 1.27 1.27)) hide)
     )
@@
       (effects (font (size 1.27 1.27)) (justify left))
     )
-    (property "Value" "LMV331" (at 524.51 251.46 0)
+    (property "Value" "MCP6456U" (at 524.51 251.46 0)
       (effects (font (size 1.27 1.27)) (justify left))
     )
@@
       (effects (font (size 1.27 1.27)) hide)
     )
-    (property "Datasheet" "http://www.ti.com/lit/ds/symlink/lmv331.pdf" (at 524.51 250.19 0)
+    (property "Datasheet" "https://ww1.microchip.com/downloads/aemDocuments/documents/MSLD/ProductDocuments/DataSheets/MCP6546-Open-Drain-Output-Sub-Microamp-Comparators-DS20001714.pdf" (at 524.51 250.19 0)
       (effects (font (size 1.27 1.27)) hide)
     )

Commit message: * Add power indicator LED to front panel
Parts:
- added LED5: LED, LED_SMD:LED_LiteOn_LTST-S326, symbol Device:LED
- added R47: 1K, Resistor_SMD:R_0603_1608Metric, symbol Device:R
Connections:
- net +3V3: now also R47.2
- net GND: now also LED5.1 (K)
- new net: LED5.2 (A), R47.1
Changed lines of the file:
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@@
   (junction (at 381 349.25) (diameter 0) (color 0 0 0 0)
   )
+  (junction (at 331.47 87.63) (diameter 0) (color 0 0 0 0)
+  )
   (junction (at 74.93 76.2) (diameter 0) (color 0 0 0 0)
   )
@@
     (stroke (width 0) (type default))
   )
+  (wire (pts (xy 347.98 97.79) (xy 347.98 101.6))
+    (stroke (width 0) (type default))
+  )
   (wire (pts (xy 73.66 361.95) (xy 73.66 364.49))
     (stroke (width 0) (type default))
@@
     (stroke (width 0.1524) (type solid))
   )
+  (wire (pts (xy 347.98 109.22) (xy 347.98 113.03))
+    (stroke (width 0) (type default))
+  )
   (wire (pts (xy 73.66 372.11) (xy 73.66 374.65))
     (stroke (width 0) (type default))
@@
     (stroke (width 0.1524) (type solid))
   )
+  (wire (pts (xy 331.47 87.63) (xy 347.98 87.63))
+    (stroke (width 0) (type default))
+  )
   (wire (pts (xy 367.03 167.64) (xy 367.03 170.18))
     (stroke (width 0) (type default))
@@
     (stroke (width 0) (type default))
   )
+  (wire (pts (xy 347.98 87.63) (xy 347.98 90.17))
+    (stroke (width 0) (type default))
+  )
   (wire (pts (xy 325.12 323.85) (xy 331.47 323.85))
     (stroke (width 0.1524) (type solid))
@@
     )
   )
+  (symbol (lib_id "power:GND") (at 347.98 113.03 0) (unit 1)
+    (in_bom yes) (on_board yes) (dnp no) (fields_autoplaced)
+    (property "Reference" "#PWR014" (at 347.98 119.38 0)
+      (effects (font (size 1.27 1.27)) hide)
+    )
+    (property "Value" "GND" (at 347.98 118.11 0)
+      (effects (font (size 1.27 1.27)))
+    )
+    (property "Footprint" "" (at 347.98 113.03 0)
+      (effects (font (size 1.27 1.27)) hide)
+    )
+    (property "Datasheet" "" (at 347.98 113.03 0)
+      (effects (font (size 1.27 1.27)) hide)
+    )
+    (pin "1")
+    (instances
+      (project "emonPi3"
+        (path "/3a5f1087-1abe-4575-9313-bd86a5e03366"
+          (reference "#PWR014") (unit 1)
+        )
+      )
+    )
+  )
   (symbol (lib_name "R_1") (lib_id "Device:R") (at 486.41 93.98 90) (unit 1)
     (in_bom yes) (on_board yes) (dnp no)
@@
     )
   )
+  (symbol (lib_id "Device:R") (at 347.98 93.98 180) (unit 1)
+    (in_bom yes) (on_board yes) (dnp no)
+    (property "Reference" "R47" (at 349.25 92.71 0)
+      (effects (font (size 1.27 1.27)) (justify right top))
+    )
+    (property "Value" "1K" (at 349.25 95.25 0)
+      (effects (font (size 1.27 1.27)) (justify right top))
+    )
+    (property "Footprint" "Resistor_SMD:R_0603_1608Metric" (at 349.758 93.98 90)
+      (effects (font (size 1.27 1.27)) hide)
+    )
+    (property "Datasheet" "~" (at 347.98 93.98 0)
+      (effects (font (size 1.27 1.27)) hide)
+    )
+    (pin "1")
+    (pin "2")
+    (instances
+      (project "emonPi3"
+        (path "/3a5f1087-1abe-4575-9313-bd86a5e03366"
+          (reference "R47") (unit 1)
+        )
+      )
+    )
+  )
   (symbol (lib_id "Connector:TestPoint") (at 379.73 156.21 0) (unit 1)
     (in_bom no) (on_board yes) (dnp no) (fields_autoplaced)
@@
         )
       )
+    )
+  )
+  (symbol (lib_name "LED_1") (lib_id "Device:LED") (at 347.98 105.41 90) (unit 1)
+    (in_bom yes) (on_board yes) (dnp no) (fields_autoplaced)
+    (property "Reference" "LED5" (at 351.79 106.3625 90)
+      (effects (font (size 1.27 1.27)) (justify right))
+    )
+    (property "Value" "LED" (at 351.79 108.9025 90)
+      (effects (font (size 1.27 1.27)) (justify right))
+    )
+    (property "Footprint" "LED_SMD:LED_LiteOn_LTST-S326" (at 347.98 105.41 0)
+      (effects (font (size 1.27 1.27)) hide)
+    )
+    (property "Datasheet" "~" (at 347.98 105.41 0)
+      (effects (font (size 1.27 1.27)) hide)
+    )
+    (pin "1")
+    (pin "2")
+    (instances
+      (project "emonPi3"
+        (path "/3a5f1087-1abe-4575-9313-bd86a5e03366"
+          (reference "LED5") (unit 1)
+        )
+      )

Commit message: * LED Rationalisation
  - Combine PROG and STATUS as bicolour LED on front panel
  - Mark USER LEDs and switch as DNP, unlikely to be available in
    OEM products.
Parts:
- removed LED1, LED2: Red 1.85V, LED_SMD:LED_0805_2012Metric, symbol Device:LED
- removed LED5: LED, LED_SMD:LED_LiteOn_LTST-S326, symbol Device:LED
- removed R46, R49: 1K, Resistor_SMD:R_0603_1608Metric, symbol Device:R
- added LED5: LED_Dual_KAK, LED_SMD:LED_LiteOn_LTST-S326, symbol Device:LED_Dual_KAK
- LED3, LED4, R50, R51, R52, R53, SW2: now not fitted
Connections:
- net ~{LED_PROG}: now also LED5.1 (K1)
- net ~{LED_STATUS}: now also LED5.3 (K2)
- net at R47.1: now also LED5.2 (A)
Other:
- moved on the sheet: R47

Commit message: * Expose !RESET to Pi to allow entry to bootloader
Parts:
- removed H8: MountingHole, MountingHole:MountingHole_2.1mm, symbol Mechanical:MountingHole
Connections:
- net ~{RESET}: now also J11.17 (Pin_17)
- no-connect marks 16 -> 15
Changed lines of the file:
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@@
   (no_connect (at 419.1 334.01))
   (no_connect (at 406.4 52.07))
-  (no_connect (at 406.4 72.39))
   (no_connect (at 537.21 71.12))
   (no_connect (at 363.22 182.88))
@@
     (stroke (width 0) (type default))
   )
+  (wire (pts (xy 384.81 72.39) (xy 406.4 72.39))
+    (stroke (width 0) (type default))
+  )
   (wire (pts (xy 118.11 62.23) (xy 127 62.23))
     (stroke (width 0) (type default))
@@
     (effects (font (size 1.2446 1.2446)) (justify left bottom))
   )
+  (label "~{RESET}" (at 384.81 72.39 0) (fields_autoplaced)
+    (effects (font (size 1.27 1.27)) (justify left bottom))
+  )
   (label "P_OW_1" (at 153.67 165.1 0) (fields_autoplaced)
     (effects (font (size 1.27 1.27)) (justify left bottom))
@@
         )
       )
-    )
-  )
-  (symbol (lib_id "Mechanical:MountingHole") (at 506.73 325.12 0) (unit 1)
-    (in_bom no) (on_board yes) (dnp no) (fields_autoplaced)
-    (property "Reference" "H8" (at 509.27 324.485 0)
-      (effects (font (size 1.27 1.27)) (justify left))
-    )
-    (property "Value" "MountingHole" (at 509.27 327.025 0)
-      (effects (font (size 1.27 1.27)) (justify left))
-    )
-    (property "Footprint" "MountingHole:MountingHole_2.1mm" (at 506.73 325.12 0)
-      (effects (font (size 1.27 1.27)) hide)
-    )
-    (property "Datasheet" "~" (at 506.73 325.12 0)
-      (effects (font (size 1.27 1.27)) hide)
-    )
-    (instances
-      (project "emonPi3"
-        (path "/3a5f1087-1abe-4575-9313-bd86a5e03366"
-          (reference "H8") (unit 1)
-        )
-      )
