File: pcb/emonpi3/emonPi3.kicad_sch (KiCad schematic)
At the start: 126 parts, among them CN1 CONN_03SCREW, CN2 CONN_03SCREW, CN3 CONN_03SCREW, J10 Conn_ARM_JTAG_SWD_10, J11 Conn_02x13_Odd_Even, J12 PINHD-1X9, J7 CONN_04PTH, J8 CONN_04PTH, J9 USB_C_Receptacle_USB2.0, SW1 SW_Push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

Commit message: * Remove ANALOG_INPUT AA filter
  - Will be onboard expander board
  - Allows different use of the ANALOG_INPUT port
Parts:
- removed C9: 10n, Capacitor_SMD:C_0603_1608Metric, symbol Device:C
- removed R7: 3K3, Resistor_SMD:R_0603_1608Metric, symbol Device:R
Connections:
- net AIN_LPFILT is gone; now on net ANALOG_INPUT: U3.17 (PA08)
Changed lines of the file:
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@@
   (junction (at 372.11 323.85) (diameter 0) (color 0 0 0 0)
   )
-  (junction (at 73.66 361.95) (diameter 0) (color 0 0 0 0)
-  )
   (junction (at 374.65 175.26) (diameter 0) (color 0 0 0 0)
   )
@@
     (stroke (width 0) (type default))
   )
-  (polyline (pts (xy 12.7 350.52) (xy 135.89 350.52))
-    (stroke (width 0.1524) (type solid))
-  )
   (wire (pts (xy 317.5 116.84) (xy 317.5 120.65))
     (stroke (width 0) (type default))
@@
     (stroke (width 0) (type default))
   )
-  (wire (pts (xy 46.99 361.95) (xy 63.5 361.95))
-    (stroke (width 0) (type default))
-  )
   (wire (pts (xy 229.87 381) (xy 227.33 381))
     (stroke (width 0) (type default))
@@
     (stroke (width 0) (type default))
   )
-  (wire (pts (xy 71.12 361.95) (xy 73.66 361.95))
-    (stroke (width 0) (type default))
-  )
   (wire (pts (xy 541.02 63.5) (xy 554.99 63.5))
     (stroke (width 0) (type default))
@@
     (stroke (width 0) (type default))
   )
-  (wire (pts (xy 73.66 361.95) (xy 73.66 364.49))
-    (stroke (width 0) (type default))
-  )
   (wire (pts (xy 363.22 175.26) (xy 374.65 175.26))
     (stroke (width 0) (type default))
@@
     (stroke (width 0.1524) (type solid))
   )
-  (wire (pts (xy 73.66 372.11) (xy 73.66 374.65))
-    (stroke (width 0) (type default))
-  )
   (wire (pts (xy 346.71 226.06) (xy 346.71 228.6))
     (stroke (width 0) (type default))
@@
     (stroke (width 0) (type default))
   )
-  (wire (pts (xy 73.66 361.95) (xy 90.17 361.95))
-    (stroke (width 0) (type default))
-  )
   (wire (pts (xy 255.27 160.02) (xy 255.27 162.56))
     (stroke (width 0) (type default))
@@
     (effects (font (size 1.3513 1.3513)) (justify left bottom))
   )
-  (label "AIN_LPFILT" (at 223.52 193.04 0) (fields_autoplaced)
+  (label "ANALOG_INPUT" (at 223.52 193.04 0) (fields_autoplaced)
     (effects (font (size 1.27 1.27)) (justify left bottom))
   )
@@
     (effects (font (size 1.27 1.27)) (justify right bottom))
   )
-  (label "ANALOG_INPUT" (at 46.99 361.95 0) (fields_autoplaced)
-    (effects (font (size 1.27 1.27)) (justify left bottom))
-  )
   (label "RFM_IRQ_UC" (at 292.1 208.28 180) (fields_autoplaced)
     (effects (font (size 1.27 1.27)) (justify right bottom))
@@
     (effects (font (size 1.27 1.27)) (justify right bottom))
   )
-  (label "AIN_LPFILT" (at 90.17 361.95 180) (fields_autoplaced)
-    (effects (font (size 1.27 1.27)) (justify right bottom))
-  )
   (label "P_OW_1" (at 223.52 213.36 0) (fields_autoplaced)
     (effects (font (size 1.2446 1.2446)) (justify left bottom))
@@
     )
   )
-  (symbol (lib_id "Device:C") (at 73.66 368.3 0) (unit 1)
-    (in_bom yes) (on_board yes) (dnp no)
-    (property "Reference" "C9" (at 76.2 367.03 0)
-      (effects (font (size 1.27 1.27)) (justify left bottom))
-    )
-    (property "Value" "10n" (at 76.2 369.57 0)
-      (effects (font (size 1.27 1.27)) (justify left bottom))
-    )
-    (property "Footprint" "Capacitor_SMD:C_0603_1608Metric" (at 74.6252 372.11 0)
-      (effects (font (size 1.27 1.27)) hide)
-    )
-    (property "Datasheet" "~" (at 73.66 368.3 0)
-      (effects (font (size 1.27 1.27)) hide)
-    )
-    (pin "1")
-    (pin "2")
-    (instances
-      (project "emonPi3"
-        (path "/3a5f1087-1abe-4575-9313-bd86a5e03366"
-          (reference "C9") (unit 1)
-        )
-      )
-    )
-  )
   (symbol (lib_id "Device:R") (at 510.54 278.13 0) (mirror y) (unit 1)
     (in_bom yes) (on_board yes) (dnp no)
@@
     )
   )
-  (symbol (lib_id "power:GND") (at 73.66 374.65 0) (unit 1)
-    (in_bom yes) (on_board yes) (dnp no) (fields_autoplaced)
-    (property "Reference" "#PWR06" (at 73.66 381 0)
-      (effects (font (size 1.27 1.27)) hide)
-    )
-    (property "Value" "GND" (at 73.66 379.73 0)
-      (effects (font (size 1.27 1.27)))
-    )
-    (property "Footprint" "" (at 73.66 374.65 0)
-      (effects (font (size 1.27 1.27)) hide)
-    )
-    (property "Datasheet" "" (at 73.66 374.65 0)
-      (effects (font (size 1.27 1.27)) hide)
-    )
-    (pin "1")
-    (instances
-      (project "emonPi3"
-        (path "/3a5f1087-1abe-4575-9313-bd86a5e03366"
-          (reference "#PWR06") (unit 1)
-        )
-      )
-    )
-  )
   (symbol (lib_id "power:GND") (at 185.42 327.66 0) (unit 1)
     (in_bom yes) (on_board yes) (dnp no) (fields_autoplaced)
@@
         )
       )
-    )
-  )
-  (symbol (lib_id "Device:R") (at 67.31 361.95 270) (mirror x) (unit 1)
-    (in_bom yes) (on_board yes) (dnp no)
-    (property "Reference" "R7" (at 64.77 360.68 90)
-      (effects (font (size 1.27 1.27)) (justify left top))
-    )
-    (property "Value" "3K3" (at 64.77 363.22 90)
-      (effects (font (size 1.27 1.27)) (justify left bottom))
-    )
-    (property "Footprint" "Resistor_SMD:R_0603_1608Metric" (at 67.31 363.728 90)
-      (effects (font (size 1.27 1.27)) hide)
-    )
-    (property "Datasheet" "~" (at 67.31 361.95 0)
-      (effects (font (size 1.27 1.27)) hide)
-    )
-    (pin "1")
-    (pin "2")
-    (instances
-      (project "emonPi3"
-        (path "/3a5f1087-1abe-4575-9313-bd86a5e03366"
-          (reference "R7") (unit 1)
-        )
-      )

Commit message: * Split ANALOG_INPUT and CT12
  - Allows all 12 CTs to be used along with the ANALOG_INPUT
  - Removed USER LED0
Parts:
- removed LED3: Red 1.85V, LED_SMD:LED_0805_2012Metric, symbol Device:LED
- removed R51: 1K, Resistor_SMD:R_0603_1608Metric, symbol Device:R
- J10, J12, J8: now fitted
- LED5: MPN (none) -> LTST-S326KGJRKT; Manufacturer (none) -> Lite-On; Mouser (none) -> 859-LTST-S326KGJRKT
- U1: MPN (none) -> MCP1501T-10E/CHY; Manufacturer (none) -> Microchip Technology; Mouser (none) -> 579-MCP1501T-10E/CHY
- U2: MPN (none) -> USBLC6-2P6; Manufacturer (none) -> STMicroelectronics; Mouser (none) -> 511-USBLC6-2P6
- U3: MPN (none) -> ATSAMD21J17A-MU; Manufacturer (none) -> Microchip; Mouser (none) -> 556-ATSAMD21J17A-MU
- U4: MPN (none) -> AP2112K-3.3TRG1; Manufacturer (none) -> Diodes Incorporated; Mouser (none) -> 621-AP2112K-3.3TRG1
- U5: value ~ -> TPS2116; MPN (none) -> TPS2116DRLR; Manufacturer (none) -> TI; Mouser (none) -> 595-TPS2116DRLR
- U6: value MCP6456U -> MCP6546U; MPN (none) -> MCP6546U-E/OT; Manufacturer (none) -> Microchip; Mouser (none) -> 579-MCP6546UT-E/OT
- U8: value 24AA02-OT -> 24FC08-OT; MPN (none) -> 24FC08T-I/OT; Manufacturer (none) -> Microchip; Mouser (none) -> 579-24FC08T-I/OT
Connections:
- net ~{LED_USER0} is gone; now on net ~{USER_BUTTON}: U3.23 (PB10)
- net ANALOG_INPUT: now also U3.18 (PA09); no longer J12.4 (Pin_4), U3.17 (PA08)
- net VCAL_{HIGH}: now also U3.19 (PA10); no longer U3.18 (PA09)
- net VCAL_{LOW}: now also U3.20 (PA11); no longer U3.19 (PA10)
- net ~{USER_BUTTON}: no longer U3.20 (PA11)
- new net CT12: J12.4 (Pin_4), U3.17 (PA08)
Other:
- note added: "Raspberry Pi Header"
- note removed: "Rasperry Pi Header"
