File: pcb/6ct-expander/6ct-expander.kicad_sch (KiCad schematic)
At the start: 3 parts, among them J13 Conn_02x05_Odd_Even

Commit message: [6CT] Finalise CT expander board
Parts:
- renumbered H4 to H1, H4 to H2, J13 to J7
