File: pcb/6ct-expander/6ct-expander.kicad_pcb (KiCad board)
At the start: 2 copper layers, 88 x 30 mm, 57 parts, among them J1 SJ-3524-SMT-TR, J2 SJ-3524-SMT-TR, J3 SJ-3524-SMT-TR, J4 SJ-3524-SMT-TR, J5 SJ-3524-SMT-TR, J6 SJ-3524-SMT-TR, J7 Conn_02x05_Odd_Even

Commit message: [6CT] Finalise CT expander board
Other:
- board text added: "CT Expander v1.0 - OEM 2025 github.com/awjlogan/emon32 openenergymonitor.org"
- board text removed: "CT Expander - OEM 2024 github.com/awjlogan/emon32 openenergymonitor.org"

Commit message: Freeze for manufacture
Routing:
- net Net-(D5-A2): track 7.04 -> 10.6 mm
