File: pcb/6ct-expander/6ct-expander.kicad_pcb (KiCad board)
At the start: 2 copper layers, 30 x 88 mm, 60 parts, among them J1 SJ-3524-SMT-TR, J2 SJ-3524-SMT-TR, J3 SJ-3524-SMT-TR, J4 SJ-3524-SMT-TR, J5 SJ-3524-SMT-TR, J6 SJ-3524-SMT-TR, J7 Conn_02x05_Odd_Even, J8 Conn_01x01, J9 Conn_01x01

Commit message: [CT Expander] Add missing trace on CT12
  - Added missing connection from CT12 to bias network.
Routing:
- net Net-(D5-A2): track 7.04 -> 10.6 mm
- net /V_{REF}: track 79.2 -> 77.2 mm
- net /CT10: track 13.0 -> 12.0 mm
Other:
- board text added: "CT Expander v1.1 - OEM 2026 openenergymonitor.org"
- board text removed: "CT Expander v1.0 - OEM 2026 openenergymonitor.org"
Changed lines of the file:
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@@
 	(title_block
 		(title "OEM 6CT expander")
-		(date "2026-05-06")
-		(rev "v1.0")
+		(date "2026-07-20")
+		(rev "v1.1")
 		(company "OpenEnergyMonitor")
 	)
@@
 		(layer "Edge.Cuts")
 	)
-	(gr_text "CT Expander v1.0 - OEM 2026\nopenenergymonitor.org"
+	(gr_text "CT Expander v1.1 - OEM 2026\nopenenergymonitor.org"
 		(at 130.5 55.5 0)
 		(layer "F.SilkS")
@@
 	(segment
 		(start 146.3 98.3)
-		(end 146.5 98.5)
+		(end 147.275 99.275)
 		(width 0.3)
 		(layer "F.Cu")
@@
 	)
 	(segment
-		(start 147.275 99.275)
-		(end 146.5 98.5)
-		(width 0.3)
-		(layer "F.Cu")
-		(net 7)
-	)
-	(segment
 		(start 145 98.3)
 		(end 144.2 98.3)
@@
 	(segment
 		(start 152.165 99.335)
-		(end 152.5 99)
-		(width 0.3)
-		(layer "F.Cu")
-		(net 9)
-	)
-	(segment
-		(start 152.165 99.335)
 		(end 153.834 97.666)
 		(width 0.3)
@@
 	)
 	(segment
-		(start 152.5 99)
-		(end 152.505 99.005)
-		(width 0.3)
-		(layer "F.Cu")
-		(net 9)
-	)
-	(segment
 		(start 153.834 97.666)
 		(end 155.426 97.666)
@@
 	)
 	(segment
-		(start 152.5 101)
-		(end 153.155 100.345)
-		(width 0.3)
-		(layer "F.Cu")
-		(net 12)
-	)
-	(segment
 		(start 153 108.175)
 		(end 153 106.5)
@@
 	)
 	(segment
-		(start 152.5 101)
-		(end 152.5 100.73)
-		(width 0.3)
-		(layer "F.Cu")
-		(net 12)
-	)
-	(segment
 		(start 152.5 106)
-		(end 152.5 101)
+		(end 152.5 100.73)
 		(width 0.3)
 		(layer "F.Cu")
@@
 	)
 	(segment
+		(start 141.8 135.7)
+		(end 141.8 138.3375)
+		(width 0.3)
+		(layer "F.Cu")
+		(net 16)
+	)
+	(segment
 		(start 145 138.3)
 		(end 144.2 138.3)
@@
 	)
 	(segment
+		(start 141.8 138.3375)
+		(end 142.4625 139)
+		(width 0.3)
+		(layer "F.Cu")
+		(net 16)
+	)
+	(segment
 		(start 151 136.175)
 		(end 149.05 136.175)
@@
 	)
 	(segment
-		(start 156.765 86.5)
+		(start 156.765 77.265)
 		(end 156.765 87.735)
 		(width 0.3)
@@
 	)
 	(segment
-		(start 156.765 86.5)
-		(end 156.765 77.265)
-		(width 0.3)
-		(layer "F.Cu")
-		(net 18)
-	)
-	(segment
 		(start 155 69.775)
 		(end 153.05 69.775)
@@
 	)
 	(segment
-		(start 150 97.5)
-		(end 149 97.5)
+		(start 149 97.5)
+		(end 153.19 97.5)
 		(width 0.5)
 		(layer "B.Cu")
@@
 	)
 	(segment
-		(start 150 97.5)
-		(end 153.19 97.5)
-		(width 0.5)
-		(layer "B.Cu")
-		(net 26)
-	)
-	(segment
 		(start 149 120)
 		(end 149 131.5)
@@
 		(width 0.5)
 		(layer "B.Cu")
-		(net 26)
-	)
-	(segment
-		(start 152 97.5)
-		(end 150 97.5)
-		(width 0.5)
-		(layer "B.Cu")
