File: pcb/6ct-expander/ct_frontend.kicad_sch (KiCad schematic)
At the start: 9 parts, among them J1 SJ-3524-SMT-TR

Commit message: [6CT] Correct header, add extra GND pads
Parts:
- R1: LCSC C25345 -> C2107438
Other:
- title: emonPi3 / Tx6 6CT expander -> emonPi3
Changed lines of the file:
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@@
 	(paper "A4")
 	(title_block
-		(title "emonPi3 / Tx6 6CT expander")
-		(date "2025-12-10")
-		(rev "v1.1")
+		(title "emonPi3")
+		(date "2026-05-06")
+		(rev "v0.2")
 		(company "OpenEnergyMonitor / Tilt Ltd")
-		(comment 1 "Angus Logan, 2025")
+		(comment 1 "Original design: Trystan Lea & Glynn Hudson")
 		(comment 2 "Commit hash: gitrev")
 	)
@@
 			)
 		)
-		(property "LCSC" "C25345"
+		(property "LCSC" "C2107438"
 			(at 115.57 90.17 0)
 			(effects
