File: pcb/6ct-expander/ct_frontend.kicad_sch (KiCad schematic)
At the start: 9 parts, among them J1 SJ-3524-SMT-TR

Commit message: [CT Expander] Add missing trace on CT12
  - Added missing connection from CT12 to bias network.
Other:
- title: emonPi3 -> CT Expander
Changed lines of the file:
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@@
 	(paper "A4")
 	(title_block
-		(title "emonPi3")
-		(date "2026-05-06")
-		(rev "v0.2")
+		(title "CT Expander")
+		(date "2026-07-20")
+		(rev "v1.1")
 		(company "OpenEnergyMonitor / Tilt Ltd")
 		(comment 1 "Original design: Trystan Lea & Glynn Hudson")
